File: kicad/AART_Remora_12.kicad_sch (KiCad schematic)
At the start: 30 parts, among them Q1 FMMT718, Q2 EMZ1T2R, Q3 MMBFJ309, Q4 JMSL0302AU, U1 AP3015KTR-G1, U2 AP2210K-3.3TRG1

Commit message: Updated foot prints and 3d
Parts:
- L1: footprint AART11footprints:IND-SMD_L2.0-W1.6 -> AART12Footprints:IND-SMD_L2.0-W1.6
- Q4: footprint AART11footprints:DFN-8_L3.2-W3.1-P0.65-LS3.4-BL -> AART12Footprints:DFN-8_L3.2-W3.1-P0.65-LS3.4-BL
Changed lines of the file:
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@@
 		)
 		(instances
-			(project "AART11"
+			(project "AART_Remora_12"
 				(path "/4f304c91-8ecc-460d-913e-dab1ef2fd784"
 					(reference "R3")
@@
 		)
 		(instances
-			(project "AART11"
+			(project "AART_Remora_12"
 				(path "/4f304c91-8ecc-460d-913e-dab1ef2fd784"
 					(reference "#FLG01")
@@
 			)
 		)
-		(property "Footprint" "AART11footprints:DFN-8_L3.2-W3.1-P0.65-LS3.4-BL"
+		(property "Footprint" "AART12Footprints:DFN-8_L3.2-W3.1-P0.65-LS3.4-BL"
 			(at 65.405 91.44 0)
 			(hide yes)
@@
 				)
 			)
-			(project "AART11"
+			(project "AART_Remora_12"
 				(path "/4f304c91-8ecc-460d-913e-dab1ef2fd784"
 					(reference "Q4")
@@
 		)
 		(instances
-			(project "AART11"
+			(project "AART_Remora_12"
 				(path "/4f304c91-8ecc-460d-913e-dab1ef2fd784"
 					(reference "D2")
@@
 		)
 		(instances
-			(project "AART11"
+			(project "AART_Remora_12"
 				(path "/4f304c91-8ecc-460d-913e-dab1ef2fd784"
 					(reference "#PWR05")
@@
 		)
 		(instances
-			(project "AART11"
+			(project "AART_Remora_12"
 				(path "/4f304c91-8ecc-460d-913e-dab1ef2fd784"
 					(reference "#FLG02")
@@
 		)
 		(instances
-			(project "AART11"
+			(project "AART_Remora_12"
 				(path "/4f304c91-8ecc-460d-913e-dab1ef2fd784"
 					(reference "R2")
@@
 		)
 		(instances
-			(project "AART11"
+			(project "AART_Remora_12"
 				(path "/4f304c91-8ecc-460d-913e-dab1ef2fd784"
 					(reference "#PWR08")
@@
 		)
 		(instances
-			(project "AART11"
+			(project "AART_Remora_12"
 				(path "/4f304c91-8ecc-460d-913e-dab1ef2fd784"
 					(reference "#PWR07")
@@
 		)
 		(instances
-			(project "AART11"
+			(project "AART_Remora_12"
 				(path "/4f304c91-8ecc-460d-913e-dab1ef2fd784"
 					(reference "U2")
@@
 		)
 		(instances
-			(project "AART11"
+			(project "AART_Remora_12"
 				(path "/4f304c91-8ecc-460d-913e-dab1ef2fd784"
 					(reference "C6")
@@
 		)
 		(instances
-			(project "AART11"
+			(project "AART_Remora_12"
 				(path "/4f304c91-8ecc-460d-913e-dab1ef2fd784"
 					(reference "#PWR09")
@@
 		)
 		(instances
-			(project "AART11"
+			(project "AART_Remora_12"
 				(path "/4f304c91-8ecc-460d-913e-dab1ef2fd784"
 					(reference "R7")
@@
 		)
 		(instances
-			(project "AART11"
+			(project "AART_Remora_12"
 				(path "/4f304c91-8ecc-460d-913e-dab1ef2fd784"
 					(reference "#PWR04")
@@
 		)
 		(instances
-			(project "AART11"
+			(project "AART_Remora_12"
 				(path "/4f304c91-8ecc-460d-913e-dab1ef2fd784"
 					(reference "Q2")
@@
 		)
 		(instances
-			(project "AART11"
+			(project "AART_Remora_12"
 				(path "/4f304c91-8ecc-460d-913e-dab1ef2fd784"
 					(reference "TP2")
@@
 		)
 		(instances
-			(project "AART11"
+			(project "AART_Remora_12"
 				(path "/4f304c91-8ecc-460d-913e-dab1ef2fd784"
 					(reference "#FLG03")
@@
 		)
 		(instances
-			(project "AART11"
+			(project "AART_Remora_12"
 				(path "/4f304c91-8ecc-460d-913e-dab1ef2fd784"
 					(reference "TP5")
@@
 		)
 		(instances
-			(project "AART11"
+			(project "AART_Remora_12"
 				(path "/4f304c91-8ecc-460d-913e-dab1ef2fd784"
 					(reference "#FLG04")
@@
 		)
 		(instances
-			(project "AART11"
+			(project "AART_Remora_12"
 				(path "/4f304c91-8ecc-460d-913e-dab1ef2fd784"
 					(reference "C2")
@@
 		)
 		(instances
-			(project "AART11"
+			(project "AART_Remora_12"
 				(path "/4f304c91-8ecc-460d-913e-dab1ef2fd784"
 					(reference "#PWR06")
@@
 		)
 		(instances
-			(project "AART11"
+			(project "AART_Remora_12"
 				(path "/4f304c91-8ecc-460d-913e-dab1ef2fd784"
 					(reference "R8")
@@
 		)
 		(instances
-			(project "AART11"
+			(project "AART_Remora_12"
 				(path "/4f304c91-8ecc-460d-913e-dab1ef2fd784"
 					(reference "GND1")
@@
 		)
 		(instances
-			(project "AART11"
+			(project "AART_Remora_12"
 				(path "/4f304c91-8ecc-460d-913e-dab1ef2fd784"
 					(reference "R5")
@@
 		)
 		(instances
-			(project "AART11"
+			(project "AART_Remora_12"
 				(path "/4f304c91-8ecc-460d-913e-dab1ef2fd784"
 					(reference "TP1")
@@
 		)
 		(instances
-			(project "AART11"
+			(project "AART_Remora_12"
 				(path "/4f304c91-8ecc-460d-913e-dab1ef2fd784"
 					(reference "C1")
@@
 		)
 		(instances
-			(project "AART11"
+			(project "AART_Remora_12"
 				(path "/4f304c91-8ecc-460d-913e-dab1ef2fd784"
 					(reference "#PWR010")
@@
 		)
 		(instances
-			(project "AART11"
+			(project "AART_Remora_12"
 				(path "/4f304c91-8ecc-460d-913e-dab1ef2fd784"
 					(reference "C4")
@@
 		)
 		(instances
-			(project "AART11"
+			(project "AART_Remora_12"
 				(path "/4f304c91-8ecc-460d-913e-dab1ef2fd784"
 					(reference "C3")
@@
 		)
 		(instances
-			(project "AART11"
+			(project "AART_Remora_12"
 				(path "/4f304c91-8ecc-460d-913e-dab1ef2fd784"
 					(reference "R6")
@@
 		)
 		(instances
-			(project "AART11"
+			(project "AART_Remora_12"
 				(path "/4f304c91-8ecc-460d-913e-dab1ef2fd784"
 					(reference "D1")
@@
 		)
 		(instances
-			(project "AART11"
+			(project "AART_Remora_12"
 				(path "/4f304c91-8ecc-460d-913e-dab1ef2fd784"
 					(reference "C5")
@@
 		)
 		(instances
-			(project "AART11"
+			(project "AART_Remora_12"
 				(path "/4f304c91-8ecc-460d-913e-dab1ef2fd784"
 					(reference "R1")
@@
 		)
 		(instances
-			(project "AART11"
+			(project "AART_Remora_12"
 				(path "/4f304c91-8ecc-460d-913e-dab1ef2fd784"
 					(reference "Q1")
@@
 		)
 		(instances
-			(project "AART11"
+			(project "AART_Remora_12"
 				(path "/4f304c91-8ecc-460d-913e-dab1ef2fd784"
 					(reference "#PWR03")
@@
 		)
 		(instances
-			(project "AART11"
+			(project "AART_Remora_12"
 				(path "/4f304c91-8ecc-460d-913e-dab1ef2fd784"
 					(reference "R4")
@@
 		)
 		(instances
-			(project "AART11"
+			(project "AART_Remora_12"
 				(path "/4f304c91-8ecc-460d-913e-dab1ef2fd784"
 					(reference "#PWR02")
@@
 		)
 		(instances
-			(project "AART11"
+			(project "AART_Remora_12"
 				(path "/4f304c91-8ecc-460d-913e-dab1ef2fd784"
 					(reference "Q2")
@@
 			)
 		)
-		(property "Footprint" "AART11footprints:IND-SMD_L2.0-W1.6"
+		(property "Footprint" "AART12Footprints:IND-SMD_L2.0-W1.6"
 			(at 69.85 114.3 0)
 			(hide yes)
@@
 		)
 		(instances
-			(project "AART11"
+			(project "AART_Remora_12"
 				(path "/4f304c91-8ecc-460d-913e-dab1ef2fd784"
 					(reference "L1")
@@
 		)
 		(instances
-			(project "AART11"
+			(project "AART_Remora_12"
 				(path "/4f304c91-8ecc-460d-913e-dab1ef2fd784"
 					(reference "D4")
@@
 		)
 		(instances
-			(project "AART11"
+			(project "AART_Remora_12"
 				(path "/4f304c91-8ecc-460d-913e-dab1ef2fd784"
 					(reference "#FLG05")
@@
 		)
 		(instances
-			(project "AART11"
+			(project "AART_Remora_12"
 				(path "/4f304c91-8ecc-460d-913e-dab1ef2fd784"
 					(reference "Q3")
@@
 		)
 		(instances
-			(project "AART11"
+			(project "AART_Remora_12"
 				(path "/4f304c91-8ecc-460d-913e-dab1ef2fd784"
 					(reference "D3")
@@
 		)
 		(instances
-			(project "AART11"
+			(project "AART_Remora_12"
 				(path "/4f304c91-8ecc-460d-913e-dab1ef2fd784"
 					(reference "#PWR011")
@@
 		)
 		(instances
-			(project "AART11"
+			(project "AART_Remora_12"
 				(path "/4f304c91-8ecc-460d-913e-dab1ef2fd784"
 					(reference "U1")
@@
 		)
 		(instances
-			(project "AART11"
+			(project "AART_Remora_12"
 				(path "/4f304c91-8ecc-460d-913e-dab1ef2fd784"
 					(reference "TP3")
@@
 		)
 		(instances
-			(project "AART11"
+			(project "AART_Remora_12"
 				(path "/4f304c91-8ecc-460d-913e-dab1ef2fd784"
 					(reference "D2")
@@
 		)
 		(instances
-			(project "AART11"
+			(project "AART_Remora_12"
 				(path "/4f304c91-8ecc-460d-913e-dab1ef2fd784"
 					(reference "D2")
@@
 		)
 		(instances
-			(project "AART11"
+			(project "AART_Remora_12"
 				(path "/4f304c91-8ecc-460d-913e-dab1ef2fd784"
 					(reference "#PWR01")
@@
 		)
 		(instances
-			(project "AART11"
+			(project "AART_Remora_12"
 				(path "/4f304c91-8ecc-460d-913e-dab1ef2fd784"
 					(page "3")
@@
 		)
 		(instances
-			(project "AART11"
+			(project "AART_Remora_12"
 				(path "/4f304c91-8ecc-460d-913e-dab1ef2fd784"
 					(page "2")
