File: kicad/s001.kicad_sch (KiCad schematic)
At the start: 39 parts, among them J10 Conn_01x01_Pin, J11 Conn_01x01_Pin, J2 Conn_01x01_Pin, J3 Conn_01x01_Pin, J8 Conn_01x01_Pin, J9 Conn_01x01_Pin, Q10 JMSL0302AU, Q5 JMSL0302AU, Q6 JMSL0302AU, Q7 JMSL0302AU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

Commit message: Updated foot prints and 3d
Parts:
- C11, C12, C13, C14, C15, C16, C17, C18, C19, C20: footprint AART11footprints:C_0805_2012Metric_22µF -> AART12Footprints:C_0805_2012Metric_22µF
- Q10, Q5, Q6, Q7, Q8, Q9: footprint AART11footprints:DFN-8_L3.2-W3.1-P0.65-LS3.4-BL -> AART12Footprints:DFN-8_L3.2-W3.1-P0.65-LS3.4-BL
