File: kicad/s002.kicad_sch (KiCad schematic)
At the start: 13 parts, among them J1 Conn_01x01_Pin, J4 Conn_01x04, J5 Conn_01x01, J6 Conn_01x01, J7 Conn_01x01, U4 AT32F421G8U7

Commit message: Updated foot prints and 3d
Parts:
- J4: footprint AART11footprints:HDG 1x04 P0.6 Horizontal -> AART12Footprints:HDG 1x04 P0.6 Horizontal
- U4: footprint AART11footprints:QFN-28_L4.0-W4.0-P0.40-TL-EP2.4 -> AART12Footprints:QFN-28_L4.0-W4.0-P0.40-TL-EP2.4
Changed lines of the file:
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@@
 		)
 		(instances
-			(project "AART11"
+			(project "AART_Remora_12"
 				(path "/4f304c91-8ecc-460d-913e-dab1ef2fd784/3bfdbefe-78b2-4ffd-b0a6-b186bb5b1312"
 					(reference "R19")
@@
 		)
 		(instances
-			(project "AART11"
+			(project "AART_Remora_12"
 				(path "/4f304c91-8ecc-460d-913e-dab1ef2fd784/3bfdbefe-78b2-4ffd-b0a6-b186bb5b1312"
 					(reference "#PWR019")
@@
 		)
 		(instances
-			(project "AART11"
+			(project "AART_Remora_12"
 				(path "/4f304c91-8ecc-460d-913e-dab1ef2fd784/3bfdbefe-78b2-4ffd-b0a6-b186bb5b1312"
 					(reference "#PWR018")
@@
 			)
 		)
-		(property "Footprint" "AART11footprints:HDG 1x04 P0.6 Horizontal"
+		(property "Footprint" "AART12Footprints:HDG 1x04 P0.6 Horizontal"
 			(at 254 55.88 0)
 			(hide yes)
@@
 		)
 		(instances
-			(project "AART11"
+			(project "AART_Remora_12"
 				(path "/4f304c91-8ecc-460d-913e-dab1ef2fd784/3bfdbefe-78b2-4ffd-b0a6-b186bb5b1312"
 					(reference "J4")
@@
 		)
 		(instances
-			(project "AART11"
+			(project "AART_Remora_12"
 				(path "/4f304c91-8ecc-460d-913e-dab1ef2fd784/3bfdbefe-78b2-4ffd-b0a6-b186bb5b1312"
 					(reference "R20")
@@
 		)
 		(instances
-			(project "AART11"
+			(project "AART_Remora_12"
 				(path "/4f304c91-8ecc-460d-913e-dab1ef2fd784/3bfdbefe-78b2-4ffd-b0a6-b186bb5b1312"
 					(reference "J7")
@@
 		)
 		(instances
-			(project "AART11"
+			(project "AART_Remora_12"
 				(path "/4f304c91-8ecc-460d-913e-dab1ef2fd784/3bfdbefe-78b2-4ffd-b0a6-b186bb5b1312"
 					(reference "#PWR017")
@@
 		)
 		(instances
-			(project "AART11"
+			(project "AART_Remora_12"
 				(path "/4f304c91-8ecc-460d-913e-dab1ef2fd784/3bfdbefe-78b2-4ffd-b0a6-b186bb5b1312"
 					(reference "R18")
@@
 		)
 		(instances
-			(project "AART11"
+			(project "AART_Remora_12"
 				(path "/4f304c91-8ecc-460d-913e-dab1ef2fd784/3bfdbefe-78b2-4ffd-b0a6-b186bb5b1312"
 					(reference "R21")
@@
 		)
 		(instances
-			(project "AART11"
+			(project "AART_Remora_12"
 				(path "/4f304c91-8ecc-460d-913e-dab1ef2fd784/3bfdbefe-78b2-4ffd-b0a6-b186bb5b1312"
 					(reference "C22")
@@
 		)
 		(instances
-			(project "AART11"
+			(project "AART_Remora_12"
 				(path "/4f304c91-8ecc-460d-913e-dab1ef2fd784/3bfdbefe-78b2-4ffd-b0a6-b186bb5b1312"
 					(reference "J6")
@@
 		)
 		(instances
-			(project "AART11"
+			(project "AART_Remora_12"
 				(path "/4f304c91-8ecc-460d-913e-dab1ef2fd784/3bfdbefe-78b2-4ffd-b0a6-b186bb5b1312"
 					(reference "C21")
@@
 			)
 		)
-		(property "Footprint" "AART11footprints:QFN-28_L4.0-W4.0-P0.40-TL-EP2.4"
+		(property "Footprint" "AART12Footprints:QFN-28_L4.0-W4.0-P0.40-TL-EP2.4"
 			(at 82.55 76.2 0)
 			(hide yes)
@@
 		)
 		(instances
-			(project "AART11"
+			(project "AART_Remora_12"
 				(path "/4f304c91-8ecc-460d-913e-dab1ef2fd784/3bfdbefe-78b2-4ffd-b0a6-b186bb5b1312"
 					(reference "U4")
@@
 		)
 		(instances
-			(project "AART11"
+			(project "AART_Remora_12"
 				(path "/4f304c91-8ecc-460d-913e-dab1ef2fd784/3bfdbefe-78b2-4ffd-b0a6-b186bb5b1312"
 					(reference "J1")
@@
 		)
 		(instances
-			(project "AART11"
+			(project "AART_Remora_12"
 				(path "/4f304c91-8ecc-460d-913e-dab1ef2fd784/3bfdbefe-78b2-4ffd-b0a6-b186bb5b1312"
 					(reference "C23")
@@
 		)
 		(instances
-			(project "AART11"
+			(project "AART_Remora_12"
 				(path "/4f304c91-8ecc-460d-913e-dab1ef2fd784/3bfdbefe-78b2-4ffd-b0a6-b186bb5b1312"
 					(reference "J5")
